File: Sensor.brd (EAGLE design)
At the start: 100 x 80 mm, 7 parts, among them U1 CNY70, U2 CNY70

Commit message: Actualizacion
Parts:
- removed U1, U2: CNY70, E&R_Sensores:CNY70
- added U$1, U$2: CNY70, cny70:4
- R1: value 10K -> 220
- R4: value 220 -> 10K
- moved R3 44.4 mm to (17.8, 5.71)
- moved R4 44.4 mm to (17.8, 10.8), turned to 180 degrees
- moved R2 38.0 mm to (17.8, 15.9), turned to 180 degrees
- moved R1 36.8 mm to (17.8, 21.0)
- moved SV1 28.0 mm to (7.62, 13.3), turned to 270 degrees
Connections:
- removed net N$1: R3.2, U1.2
- new net N$3: R3.2, U$2.K
- net GND: now also R1.1, R3.1, R4.2, SV1.2; no longer R1.2, SV1.4, U1.1, U2.1
- net N$2: now also R1.2, U$1.K; no longer R4.2, U2.2
- net S1: now also SV1.3, U$1.E; no longer SV1.1, U1.3
- net S2: now also R4.1, SV1.4, U$2.E; no longer R1.1, SV1.2, U2.3
- net VCC: now also SV1.1, U$1.A, U$1.C, U$2.A, U$2.C; no longer R3.1, R4.1, SV1.3, U1.4, U2.4
Routing:
- net VCC: track 0.00 -> 56.9 mm
- net S1: track 0.00 -> 42.3 mm
- net S2: track 0.00 -> 33.5 mm
- net GND: track 0.00 -> 20.3 mm
- net N$3: track 0.00 -> 9.09 mm
- net N$2: track 0.00 -> 5.08 mm
- added copper zone on layer 16, net N$5
Other:
- board size 100 x 80 mm -> 35 x 26.4 mm
- board text added: "S1"
- board text added: "S2"
- board text added: "SISCOM J.T.E.V 09/2017"
- board text added: "V+"
- board text added: "V-"
