File: Sensor.sch (EAGLE design)
At the start: 7 parts, among them U1 CNY70, U2 CNY70

Commit message: Actualizacion
Parts:
- removed U1, U2: CNY70, E&R_Sensores:CNY70
- added U$1, U$2: CNY70, cny70:CNY70
- R1: value 10K -> 220
- R4: value 220 -> 10K
Connections:
- removed net N$1: R3.2, U1.2
- new net N$3: R3.2, U$2.C
- net GND: now also R1.1, R3.1, R4.2, SV1.2; no longer R1.2, SV1.4, U1.1, U2.1
- net N$2: now also R1.2, U$1.C; no longer R4.2, U2.2
- net S1: now also SV1.3, U$1.EMI; no longer SV1.1, U1.3
- net S2: now also R4.1, SV1.4, U$2.EMI; no longer R1.1, SV1.2, U2.3
- net VCC: now also SV1.1, U$1.A, U$1.COL, U$2.A, U$2.COL; no longer R3.1, R4.1, SV1.3, U1.4, U2.4
Other:
- moved on the sheet: R1, R2, R3, R4
